File: HW2/HW2/HW2.brd (EAGLE design)
At the start: 160 x 100 mm, 5 parts

Commit message: sign off
Parts:
- added C1, C2, C3, C4, C5: (no value), HW2:C025-025X050
- added J1: USB-MB-H, HW2:USB-MB-H
- added R4: (no value), HW2:0207/10
- added U$1: MCP1702, HW2:TO92
- added U$2: SLIDESLIDE, HW2:SLIDE
- R1: value 10k -> (none); device resistor:0207/7 -> HW2:0207/10
- R2, R3: device resistor:0207/7 -> HW2:0207/10
- moved LED2 673.5 mm to (-50.0, -650.0)
- moved LED1 618.5 mm to (-50.0, -600.0)
- moved R3 512.4 mm to (-50.0, -500.0)
- moved R2 457.5 mm to (-50.0, -450.0)
- moved R1 402.6 mm to (-50.0, -400.0)
Connections:
- new net +5V: J1.VBUS, U$2.2
- new net N$3: LED1.A, R1.1
- net +3V3: now also C1.1, R1.2, U$1.3; no longer R1.1
- net GND: now also C2.2, J1.GND, U$1.1
- net N$1: now also C2.1, U$1.2, U$2.3; no longer LED1.A, R1.2

Commit message: check in
Parts:
- added C6, C7: 10uF, HW2:B45181B
- added U$3: PICKIT, HW2:1X05
- added U$4: PIC32MX250F128B, HW2:DIL28-3
- added U$5: OSCOSC, HW2:OSC
- C1, C2, C4: value (none) -> 0.1uF
- LED1: value (none) -> RED
- LED2: value (none) -> GREEN
- R1: value (none) -> 330
Connections:
- new net A0: U$4.2
- new net A1: U$4.3
- new net A4/LED: U$4.12
- new net B2: U$4.6
- new net B3: U$4.7
- new net B4/USER: U$4.11
- new net D+: J1.D+
- new net D-: J1.D-
- new net ID: J1.ID, U$4.14
- new net N$3: U$3.2, U$4.1
- new net N$7: U$4.9, U$5.3
- new net N$9: U$4.10, U$5.2
- new net PGC: U$3.3, U$4.5
- new net PGD: U$3.4, U$4.4
- net +3V3: now also C4.1, C6.+, U$3.5, U$4.13
- net +5V: now also U$4.15
- net GND: now also C1.2, C4.2, C6.-, U$3.1, U$4.8, U$5.1
Changed lines of the file:
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@@
 <element name="U$1" library="HW2" package="TO92" value="MCP1702" x="-50" y="-50"/>
 <element name="U$2" library="HW2" package="SLIDE" value="SLIDESLIDE" x="-50" y="-100"/>
-<element name="C1" library="HW2" package="C025-025X050" package3d_urn="urn:adsk.eagle:package:26151/1" value="" x="-50" y="-150"/>
-<element name="C2" library="HW2" package="C025-025X050" package3d_urn="urn:adsk.eagle:package:26151/1" value="" x="-50" y="-200"/>
+<element name="C1" library="HW2" package="C025-025X050" package3d_urn="urn:adsk.eagle:package:26151/1" value="0.1uF" x="-50" y="-150"/>
+<element name="C2" library="HW2" package="C025-025X050" package3d_urn="urn:adsk.eagle:package:26151/1" value="0.1uF" x="-50" y="-200"/>
 <element name="C3" library="HW2" package="C025-025X050" package3d_urn="urn:adsk.eagle:package:26151/1" value="" x="-50" y="-250"/>
-<element name="C4" library="HW2" package="C025-025X050" package3d_urn="urn:adsk.eagle:package:26151/1" value="" x="-50" y="-300"/>
+<element name="C4" library="HW2" package="C025-025X050" package3d_urn="urn:adsk.eagle:package:26151/1" value="0.1uF" x="-50" y="-300"/>
 <element name="C5" library="HW2" package="C025-025X050" package3d_urn="urn:adsk.eagle:package:26151/1" value="" x="-50" y="-350"/>
-<element name="R1" library="HW2" package="0207/10" package3d_urn="urn:adsk.eagle:package:25939/1" value="" x="-50" y="-400"/>
+<element name="R1" library="HW2" package="0207/10" package3d_urn="urn:adsk.eagle:package:25939/1" value="330" x="-50" y="-400"/>
 <element name="R2" library="HW2" package="0207/10" package3d_urn="urn:adsk.eagle:package:25939/1" value="" x="-50" y="-450"/>
 <element name="R3" library="HW2" package="0207/10" package3d_urn="urn:adsk.eagle:package:25939/1" value="" x="-50" y="-500"/>
 <element name="R4" library="HW2" package="0207/10" package3d_urn="urn:adsk.eagle:package:25939/1" value="" x="-50" y="-550"/>
-<element name="LED1" library="led" library_urn="urn:adsk.eagle:library:259" package="LED3MM" package3d_urn="urn:adsk.eagle:package:15797/1" value="" x="-50" y="-600"/>
-<element name="LED2" library="led" library_urn="urn:adsk.eagle:library:259" package="LED3MM" package3d_urn="urn:adsk.eagle:package:15797/1" value="" x="-50" y="-650"/>
+<element name="LED1" library="led" library_urn="urn:adsk.eagle:library:259" package="LED3MM" package3d_urn="urn:adsk.eagle:package:15797/1" value="RED" x="-50" y="-600"/>
+<element name="LED2" library="led" library_urn="urn:adsk.eagle:library:259" package="LED3MM" package3d_urn="urn:adsk.eagle:package:15797/1" value="GREEN" x="-50" y="-650"/>
+<element name="C6" library="HW2" package="B45181B" package3d_urn="urn:adsk.eagle:package:25794/1" value="10uF" x="-50" y="-700"/>
+<element name="C7" library="HW2" package="B45181B" package3d_urn="urn:adsk.eagle:package:25794/1" value="10uF" x="-50" y="-750"/>
+<element name="U$3" library="HW2" package="1X05" value="PICKIT" x="-50" y="-800"/>
+<element name="U$4" library="HW2" package="DIL28-3" value="PIC32MX250F128B" x="0" y="-850"/>
+<element name="U$5" library="HW2" package="OSC" value="OSCOSC" x="-50" y="-900"/>
 </elements>
 <signals>
 <signal name="+3V3">
 <contactref element="U$1" pad="3"/>
+<contactref element="R1" pad="2"/>
+<contactref element="C6" pad="+"/>
 <contactref element="C1" pad="1"/>
-<contactref element="R1" pad="2"/>
+<contactref element="U$3" pad="5"/>
+<contactref element="U$4" pad="13"/>
+<contactref element="C4" pad="1"/>
+<wire x1="-39.84" y1="-800" x2="-52.54" y2="-700" width="0" layer="19" extent="1-1"/>
+<wire x1="13.97" y1="-853.81" x2="-39.84" y2="-800" width="0" layer="19" extent="1-1"/>
+<wire x1="-44.92" y1="-400" x2="-52.54" y2="-700" width="0" layer="19" extent="1-1"/>
+<wire x1="-51.27" y1="-300" x2="-44.92" y2="-400" width="0" layer="19" extent="1-1"/>
+<wire x1="-51.27" y1="-150" x2="-51.27" y2="-300" width="0" layer="19" extent="1-1"/>
 <wire x1="-48.73" y1="-50" x2="-51.27" y2="-150" width="0" layer="19" extent="1-1"/>
-<wire x1="-44.92" y1="-400" x2="-51.27" y2="-150" width="0" layer="19" extent="1-1"/>
 </signal>
 <signal name="+5V">
 <contactref element="J1" pad="VBUS"/>
 <contactref element="U$2" pad="2"/>
+<contactref element="U$4" pad="15"/>
 <wire x1="-44.9" y1="51.6" x2="-50" y2="-100" width="0" layer="19" extent="1-1"/>
+<wire x1="16.51" y1="-846.19" x2="-50" y2="-100" width="0" layer="19" extent="1-1"/>
 </signal>
 <signal name="GND">
@@
 <contactref element="C2" pad="2"/>
 <contactref element="LED1" pad="K"/>
-<wire x1="-51.27" y1="-50" x2="-48.73" y2="-200" width="0" layer="19" extent="1-1"/>
+<contactref element="C6" pad="-"/>
+<contactref element="C1" pad="2"/>
+<contactref element="U$3" pad="1"/>
+<contactref element="U$5" pad="1"/>
+<contactref element="U$4" pad="8"/>
+<contactref element="C4" pad="2"/>
+<wire x1="-48.73" y1="-150" x2="-48.73" y2="-200" width="0" layer="19" extent="1-1"/>
+<wire x1="-48.73" y1="-300" x2="-48.73" y2="-200" width="0" layer="19" extent="1-1"/>
+<wire x1="-51.27" y1="-50" x2="-48.73" y2="-150" width="0" layer="19" extent="1-1"/>
 <wire x1="-44.9" y1="48.4" x2="-51.27" y2="-50" width="0" layer="19" extent="1-1"/>
-<wire x1="-48.73" y1="-600" x2="-48.73" y2="-200" width="0" layer="19" extent="1-1"/>
+<wire x1="-48.73" y1="-600" x2="-48.73" y2="-300" width="0" layer="19" extent="1-1"/>
+<wire x1="-47.46" y1="-700" x2="-48.73" y2="-600" width="0" layer="19" extent="1-1"/>
+<wire x1="-50" y1="-800" x2="-47.46" y2="-700" width="0" layer="19" extent="1-1"/>
+<wire x1="1.27" y1="-853.81" x2="-50" y2="-800" width="0" layer="19" extent="1-1"/>
+<wire x1="-52.54" y1="-900" x2="1.27" y2="-853.81" width="0" layer="19" extent="1-1"/>
 </signal>
 <signal name="N$1">
@@
 <wire x1="-50" y1="-48.095" x2="-48" y2="-100" width="0" layer="19" extent="1-1"/>
 </signal>
-<signal name="N$3">
+<signal name="N$2">
 <contactref element="R1" pad="1"/>
 <contactref element="LED1" pad="A"/>
 <wire x1="-51.27" y1="-600" x2="-55.08" y2="-400" width="0" layer="19" extent="1-1"/>
 </signal>
+<signal name="ID">
+<contactref element="J1" pad="ID"/>
+<contactref element="U$4" pad="14"/>
+<wire x1="-46.1" y1="49.2" x2="16.51" y2="-853.81" width="0" layer="19" extent="1-1"/>
+</signal>
+<signal name="D+">
+<contactref element="J1" pad="D+"/>
+</signal>
+<signal name="D-">
+<contactref element="J1" pad="D-"/>
+</signal>
+<signal name="N$3">
+<contactref element="U$3" pad="2"/>
+<contactref element="U$4" pad="1"/>
+<wire x1="-47.46" y1="-800" x2="-16.51" y2="-853.81" width="0" layer="19" extent="1-1"/>
+</signal>
+<signal name="PGD">
+<contactref element="U$3" pad="4"/>
+<contactref element="U$4" pad="4"/>
+<wire x1="-42.38" y1="-800" x2="-8.89" y2="-853.81" width="0" layer="19" extent="1-1"/>
+</signal>
+<signal name="PGC">
+<contactref element="U$3" pad="3"/>
+<contactref element="U$4" pad="5"/>
+<wire x1="-44.92" y1="-800" x2="-6.35" y2="-853.81" width="0" layer="19" extent="1-1"/>
+</signal>
+<signal name="A0">
+<contactref element="U$4" pad="2"/>
+</signal>
+<signal name="A1">
+<contactref element="U$4" pad="3"/>
+</signal>
+<signal name="B2">
+<contactref element="U$4" pad="6"/>
+</signal>
+<signal name="B3">
+<contactref element="U$4" pad="7"/>
+</signal>
+<signal name="N$7">
+<contactref element="U$4" pad="9"/>
+<contactref element="U$5" pad="3"/>
+<wire x1="3.81" y1="-853.81" x2="-47.46" y2="-900" width="0" layer="19" extent="1-1"/>
+</signal>
+<signal name="N$9">
+<contactref element="U$4" pad="10"/>
+<contactref element="U$5" pad="2"/>
+<wire x1="6.35" y1="-853.81" x2="-50" y2="-900" width="0" layer="19" extent="1-1"/>
+</signal>
+<signal name="B4/USER">
+<contactref element="U$4" pad="11"/>
+</signal>
+<signal name="A4/LED">
+<contactref element="U$4" pad="12"/>
+</signal>
 </signals>

Commit message: schem update
Parts:
- removed C5: (no value), HW2:C025-025X050
- added RESET, U$6: PB, HW2:PB
- C3: value (none) -> 1uF
- R2: value (none) -> 10k
Connections:
- new net B13: U$4.24
- new net B14: U$4.25
- new net B15: U$4.26
- new net B7: U$4.16
- new net B8: U$4.17
- new net B9: U$4.18
- new net N$13: C7.+, U$4.20
- new net N$4: LED2.K, R3.2
- net +3V3: now also C3.1, R2.2, U$4.23
- net A4/LED: now also LED2.A
- net D+: now also U$4.21
- net D-: now also U$4.22
- net GND: now also C3.2, C7.-, R3.1, RESET.2, U$4.19, U$4.27
- net N$3: now also R2.1, RESET.1
Other:
- board size 160 x 100 mm -> 50 x 50 mm
Changed lines of the file:
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@@
 <setting verticaltext="up"/>
 </settings>
-<grid distance="50" unitdist="mm" unit="mm" style="lines" multiple="1" display="yes" altdistance="50" altunitdist="mm" altunit="mm"/>
+<grid distance="1" unitdist="inch" unit="inch" style="lines" multiple="1" display="yes" altdistance="0.1" altunitdist="mm" altunit="mm"/>
 <layers>
 <layer number="1" name="Top" color="4" fill="1" visible="yes" active="yes"/>
@@
 <board>
 <plain>
-<wire x1="0" y1="0" x2="160" y2="0" width="0" layer="20"/>
-<wire x1="160" y1="0" x2="160" y2="100" width="0" layer="20"/>
-<wire x1="160" y1="100" x2="0" y2="100" width="0" layer="20"/>
-<wire x1="0" y1="100" x2="0" y2="0" width="0" layer="20"/>
+<wire x1="0" y1="0" x2="50" y2="0" width="0" layer="20"/>
+<wire x1="50" y1="0" x2="50" y2="50" width="0" layer="20"/>
+<wire x1="50" y1="50" x2="0" y2="50" width="0" layer="20"/>
+<wire x1="0" y1="50" x2="0" y2="0" width="0" layer="20"/>
 </plain>
 <attributes>
@@
 <element name="C1" library="HW2" package="C025-025X050" package3d_urn="urn:adsk.eagle:package:26151/1" value="0.1uF" x="-50" y="-150"/>
 <element name="C2" library="HW2" package="C025-025X050" package3d_urn="urn:adsk.eagle:package:26151/1" value="0.1uF" x="-50" y="-200"/>
-<element name="C3" library="HW2" package="C025-025X050" package3d_urn="urn:adsk.eagle:package:26151/1" value="" x="-50" y="-250"/>
+<element name="C3" library="HW2" package="C025-025X050" package3d_urn="urn:adsk.eagle:package:26151/1" value="1uF" x="-50" y="-250"/>
 <element name="C4" library="HW2" package="C025-025X050" package3d_urn="urn:adsk.eagle:package:26151/1" value="0.1uF" x="-50" y="-300"/>
-<element name="C5" library="HW2" package="C025-025X050" package3d_urn="urn:adsk.eagle:package:26151/1" value="" x="-50" y="-350"/>
 <element name="R1" library="HW2" package="0207/10" package3d_urn="urn:adsk.eagle:package:25939/1" value="330" x="-50" y="-400"/>
-<element name="R2" library="HW2" package="0207/10" package3d_urn="urn:adsk.eagle:package:25939/1" value="" x="-50" y="-450"/>
+<element name="R2" library="HW2" package="0207/10" package3d_urn="urn:adsk.eagle:package:25939/1" value="10k" x="-50" y="-450"/>
 <element name="R3" library="HW2" package="0207/10" package3d_urn="urn:adsk.eagle:package:25939/1" value="" x="-50" y="-500"/>
 <element name="R4" library="HW2" package="0207/10" package3d_urn="urn:adsk.eagle:package:25939/1" value="" x="-50" y="-550"/>
@@
 <element name="U$4" library="HW2" package="DIL28-3" value="PIC32MX250F128B" x="0" y="-850"/>
 <element name="U$5" library="HW2" package="OSC" value="OSCOSC" x="-50" y="-900"/>
+<element name="RESET" library="HW2" package="PB" value="PB" x="-50.8" y="-939.8"/>
+<element name="U$6" library="HW2" package="PB" value="PB" x="-50.8" y="-965.2"/>
 </elements>
 <signals>
@@
 <contactref element="U$4" pad="13"/>
 <contactref element="C4" pad="1"/>
+<contactref element="U$4" pad="23"/>
+<contactref element="C3" pad="1"/>
+<contactref element="R2" pad="2"/>
 <wire x1="-39.84" y1="-800" x2="-52.54" y2="-700" width="0" layer="19" extent="1-1"/>
-<wire x1="13.97" y1="-853.81" x2="-39.84" y2="-800" width="0" layer="19" extent="1-1"/>
-<wire x1="-44.92" y1="-400" x2="-52.54" y2="-700" width="0" layer="19" extent="1-1"/>
+<wire x1="-3.81" y1="-846.19" x2="-39.84" y2="-800" width="0" layer="19" extent="1-1"/>
+<wire x1="13.97" y1="-853.81" x2="-3.81" y2="-846.19" width="0" layer="19" extent="1-1"/>
+<wire x1="-44.92" y1="-450" x2="-52.54" y2="-700" width="0" layer="19" extent="1-1"/>
+<wire x1="-44.92" y1="-400" x2="-44.92" y2="-450" width="0" layer="19" extent="1-1"/>
 <wire x1="-51.27" y1="-300" x2="-44.92" y2="-400" width="0" layer="19" extent="1-1"/>
-<wire x1="-51.27" y1="-150" x2="-51.27" y2="-300" width="0" layer="19" extent="1-1"/>
+<wire x1="-51.27" y1="-250" x2="-51.27" y2="-300" width="0" layer="19" extent="1-1"/>
+<wire x1="-51.27" y1="-150" x2="-51.27" y2="-250" width="0" layer="19" extent="1-1"/>
 <wire x1="-48.73" y1="-50" x2="-51.27" y2="-150" width="0" layer="19" extent="1-1"/>
 </signal>
@@
 <contactref element="U$4" pad="8"/>
 <contactref element="C4" pad="2"/>
+<contactref element="U$4" pad="19"/>
+<contactref element="C7" pad="-"/>
+<contactref element="U$4" pad="27"/>
+<contactref element="C3" pad="2"/>
+<contactref element="RESET" pad="2"/>
+<contactref element="R3" pad="1"/>
 <wire x1="-48.73" y1="-150" x2="-48.73" y2="-200" width="0" layer="19" extent="1-1"/>
-<wire x1="-48.73" y1="-300" x2="-48.73" y2="-200" width="0" layer="19" extent="1-1"/>
+<wire x1="-48.73" y1="-250" x2="-48.73" y2="-200" width="0" layer="19" extent="1-1"/>
+<wire x1="-48.73" y1="-300" x2="-48.73" y2="-250" width="0" layer="19" extent="1-1"/>
 <wire x1="-51.27" y1="-50" x2="-48.73" y2="-150" width="0" layer="19" extent="1-1"/>
 <wire x1="-44.9" y1="48.4" x2="-51.27" y2="-50" width="0" layer="19" extent="1-1"/>
-<wire x1="-48.73" y1="-600" x2="-48.73" y2="-300" width="0" layer="19" extent="1-1"/>
+<wire x1="-55.08" y1="-500" x2="-48.73" y2="-300" width="0" layer="19" extent="1-1"/>
+<wire x1="-48.73" y1="-600" x2="-55.08" y2="-500" width="0" layer="19" extent="1-1"/>
 <wire x1="-47.46" y1="-700" x2="-48.73" y2="-600" width="0" layer="19" extent="1-1"/>
-<wire x1="-50" y1="-800" x2="-47.46" y2="-700" width="0" layer="19" extent="1-1"/>
-<wire x1="1.27" y1="-853.81" x2="-50" y2="-800" width="0" layer="19" extent="1-1"/>
-<wire x1="-52.54" y1="-900" x2="1.27" y2="-853.81" width="0" layer="19" extent="1-1"/>
+<wire x1="-47.46" y1="-750" x2="-47.46" y2="-700" width="0" layer="19" extent="1-1"/>
+<wire x1="-50" y1="-800" x2="-47.46" y2="-750" width="0" layer="19" extent="1-1"/>
+<wire x1="-13.97" y1="-846.19" x2="-50" y2="-800" width="0" layer="19" extent="1-1"/>
+<wire x1="1.27" y1="-853.81" x2="-13.97" y2="-846.19" width="0" layer="19" extent="1-1"/>
+<wire x1="6.35" y1="-846.19" x2="1.27" y2="-853.81" width="0" layer="19" extent="1-1"/>
+<wire x1="-52.54" y1="-900" x2="-13.97" y2="-846.19" width="0" layer="19" extent="1-1"/>
+<wire x1="-48.26" y1="-939.8" x2="-52.54" y2="-900" width="0" layer="19" extent="1-1"/>
 </signal>
 <signal name="N$1">
@@
 <signal name="D+">
 <contactref element="J1" pad="D+"/>
+<contactref element="U$4" pad="21"/>
+<wire x1="-44.9" y1="50" x2="1.27" y2="-846.19" width="0" layer="19" extent="1-1"/>
 </signal>
 <signal name="D-">
 <contactref element="J1" pad="D-"/>
+<contactref element="U$4" pad="22"/>
+<wire x1="-46.1" y1="50.8" x2="-1.27" y2="-846.19" width="0" layer="19" extent="1-1"/>
 </signal>
 <signal name="N$3">
 <contactref element="U$3" pad="2"/>
 <contactref element="U$4" pad="1"/>
-<wire x1="-47.46" y1="-800" x2="-16.51" y2="-853.81" width="0" layer="19" extent="1-1"/>
+<contactref element="R2" pad="1"/>
+<contactref element="RESET" pad="1"/>
+<wire x1="-47.46" y1="-800" x2="-55.08" y2="-450" width="0" layer="19" extent="1-1"/>
+<wire x1="-16.51" y1="-853.81" x2="-47.46" y2="-800" width="0" layer="19" extent="1-1"/>
+<wire x1="-53.34" y1="-939.8" x2="-16.51" y2="-853.81" width="0" layer="19" extent="1-1"/>
 </signal>
 <signal name="PGD">
@@
 <signal name="A4/LED">
 <contactref element="U$4" pad="12"/>
+<contactref element="LED2" pad="A"/>
+<wire x1="11.43" y1="-853.81" x2="-51.27" y2="-650" width="0" layer="19" extent="1-1"/>
+</signal>
+<signal name="B15">
+<contactref element="U$4" pad="26"/>
+</signal>
+<signal name="B14">
+<contactref element="U$4" pad="25"/>
+</signal>
+<signal name="B13">
+<contactref element="U$4" pad="24"/>
+</signal>
+<signal name="N$13">
+<contactref element="U$4" pad="20"/>
+<contactref element="C7" pad="+"/>
+<wire x1="-52.54" y1="-750" x2="3.81" y2="-846.19" width="0" layer="19" extent="1-1"/>
+</signal>
+<signal name="B9">
+<contactref element="U$4" pad="18"/>
+</signal>
+<signal name="B8">
+<contactref element="U$4" pad="17"/>
+</signal>
+<signal name="B7">
+<contactref element="U$4" pad="16"/>
+</signal>
+<signal name="N$4">
+<contactref element="LED2" pad="K"/>
+<contactref element="R3" pad="2"/>
+<wire x1="-44.92" y1="-500" x2="-48.73" y2="-650" width="0" layer="19" extent="1-1"/>
 </signal>
 </signals>
