File: HW2/HW2/HW2.brd (EAGLE design)
At the start: 50 x 50 mm, 20 parts, among them J1 USB-MB-H

Commit message: another update
Parts:
- added J3, J4: CONN8, HW2:1X08
- R3: value (none) -> 330
- R4: value (none) -> 10k
- renumbered U$6 to USER
Connections:
- net +3V3: now also R4.2
- net B4/USER: now also R4.1, USER.1
- net GND: now also USER.2
Changed lines of the file:
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@@
 <element name="R1" library="HW2" package="0207/10" package3d_urn="urn:adsk.eagle:package:25939/1" value="330" x="-50" y="-400"/>
 <element name="R2" library="HW2" package="0207/10" package3d_urn="urn:adsk.eagle:package:25939/1" value="10k" x="-50" y="-450"/>
-<element name="R3" library="HW2" package="0207/10" package3d_urn="urn:adsk.eagle:package:25939/1" value="" x="-50" y="-500"/>
-<element name="R4" library="HW2" package="0207/10" package3d_urn="urn:adsk.eagle:package:25939/1" value="" x="-50" y="-550"/>
+<element name="R3" library="HW2" package="0207/10" package3d_urn="urn:adsk.eagle:package:25939/1" value="330" x="-50" y="-500"/>
+<element name="R4" library="HW2" package="0207/10" package3d_urn="urn:adsk.eagle:package:25939/1" value="10k" x="-50" y="-550"/>
 <element name="LED1" library="led" library_urn="urn:adsk.eagle:library:259" package="LED3MM" package3d_urn="urn:adsk.eagle:package:15797/1" value="RED" x="-50" y="-600"/>
 <element name="LED2" library="led" library_urn="urn:adsk.eagle:library:259" package="LED3MM" package3d_urn="urn:adsk.eagle:package:15797/1" value="GREEN" x="-50" y="-650"/>
@@
 <element name="U$5" library="HW2" package="OSC" value="OSCOSC" x="-50" y="-900"/>
 <element name="RESET" library="HW2" package="PB" value="PB" x="-50.8" y="-939.8"/>
-<element name="U$6" library="HW2" package="PB" value="PB" x="-50.8" y="-965.2"/>
+<element name="USER" library="HW2" package="PB" value="PB" x="-50.8" y="-965.2"/>
+<element name="J3" library="HW2" package="1X08" value="CONN8" x="-50.8" y="-990.6"/>
+<element name="J4" library="HW2" package="1X08" value="CONN8" x="-50.8" y="-1016"/>
 </elements>
 <signals>
@@
 <contactref element="C3" pad="1"/>
 <contactref element="R2" pad="2"/>
+<contactref element="R4" pad="2"/>
 <wire x1="-39.84" y1="-800" x2="-52.54" y2="-700" width="0" layer="19" extent="1-1"/>
 <wire x1="-3.81" y1="-846.19" x2="-39.84" y2="-800" width="0" layer="19" extent="1-1"/>
 <wire x1="13.97" y1="-853.81" x2="-3.81" y2="-846.19" width="0" layer="19" extent="1-1"/>
-<wire x1="-44.92" y1="-450" x2="-52.54" y2="-700" width="0" layer="19" extent="1-1"/>
+<wire x1="-44.92" y1="-550" x2="-52.54" y2="-700" width="0" layer="19" extent="1-1"/>
+<wire x1="-44.92" y1="-450" x2="-44.92" y2="-550" width="0" layer="19" extent="1-1"/>
 <wire x1="-44.92" y1="-400" x2="-44.92" y2="-450" width="0" layer="19" extent="1-1"/>
 <wire x1="-51.27" y1="-300" x2="-44.92" y2="-400" width="0" layer="19" extent="1-1"/>
@@
 <contactref element="RESET" pad="2"/>
 <contactref element="R3" pad="1"/>
+<contactref element="USER" pad="2"/>
+<wire x1="-48.26" y1="-939.8" x2="-48.26" y2="-965.2" width="0" layer="19" extent="1-1"/>
+<wire x1="-52.54" y1="-900" x2="-48.26" y2="-939.8" width="0" layer="19" extent="1-1"/>
+<wire x1="-13.97" y1="-846.19" x2="-52.54" y2="-900" width="0" layer="19" extent="1-1"/>
+<wire x1="1.27" y1="-853.81" x2="-13.97" y2="-846.19" width="0" layer="19" extent="1-1"/>
+<wire x1="6.35" y1="-846.19" x2="1.27" y2="-853.81" width="0" layer="19" extent="1-1"/>
+<wire x1="-50" y1="-800" x2="-13.97" y2="-846.19" width="0" layer="19" extent="1-1"/>
+<wire x1="-47.46" y1="-750" x2="-50" y2="-800" width="0" layer="19" extent="1-1"/>
+<wire x1="-47.46" y1="-700" x2="-47.46" y2="-750" width="0" layer="19" extent="1-1"/>
+<wire x1="-48.73" y1="-600" x2="-47.46" y2="-700" width="0" layer="19" extent="1-1"/>
+<wire x1="-55.08" y1="-500" x2="-48.73" y2="-600" width="0" layer="19" extent="1-1"/>
+<wire x1="-48.73" y1="-300" x2="-55.08" y2="-500" width="0" layer="19" extent="1-1"/>
+<wire x1="-48.73" y1="-250" x2="-48.73" y2="-300" width="0" layer="19" extent="1-1"/>
+<wire x1="-48.73" y1="-200" x2="-48.73" y2="-250" width="0" layer="19" extent="1-1"/>
 <wire x1="-48.73" y1="-150" x2="-48.73" y2="-200" width="0" layer="19" extent="1-1"/>
-<wire x1="-48.73" y1="-250" x2="-48.73" y2="-200" width="0" layer="19" extent="1-1"/>
-<wire x1="-48.73" y1="-300" x2="-48.73" y2="-250" width="0" layer="19" extent="1-1"/>
 <wire x1="-51.27" y1="-50" x2="-48.73" y2="-150" width="0" layer="19" extent="1-1"/>
 <wire x1="-44.9" y1="48.4" x2="-51.27" y2="-50" width="0" layer="19" extent="1-1"/>
-<wire x1="-55.08" y1="-500" x2="-48.73" y2="-300" width="0" layer="19" extent="1-1"/>
-<wire x1="-48.73" y1="-600" x2="-55.08" y2="-500" width="0" layer="19" extent="1-1"/>
-<wire x1="-47.46" y1="-700" x2="-48.73" y2="-600" width="0" layer="19" extent="1-1"/>
-<wire x1="-47.46" y1="-750" x2="-47.46" y2="-700" width="0" layer="19" extent="1-1"/>
-<wire x1="-50" y1="-800" x2="-47.46" y2="-750" width="0" layer="19" extent="1-1"/>
-<wire x1="-13.97" y1="-846.19" x2="-50" y2="-800" width="0" layer="19" extent="1-1"/>
-<wire x1="1.27" y1="-853.81" x2="-13.97" y2="-846.19" width="0" layer="19" extent="1-1"/>
-<wire x1="6.35" y1="-846.19" x2="1.27" y2="-853.81" width="0" layer="19" extent="1-1"/>
-<wire x1="-52.54" y1="-900" x2="-13.97" y2="-846.19" width="0" layer="19" extent="1-1"/>
-<wire x1="-48.26" y1="-939.8" x2="-52.54" y2="-900" width="0" layer="19" extent="1-1"/>
 </signal>
 <signal name="N$1">
@@
 <signal name="B4/USER">
 <contactref element="U$4" pad="11"/>
+<contactref element="R4" pad="1"/>
+<contactref element="USER" pad="1"/>
+<wire x1="8.89" y1="-853.81" x2="-55.08" y2="-550" width="0" layer="19" extent="1-1"/>
+<wire x1="-53.34" y1="-965.2" x2="8.89" y2="-853.81" width="0" layer="19" extent="1-1"/>
 </signal>
 <signal name="A4/LED">

Commit message: sign on
Connections:
- new net N$18: J4.3
- new net N$19: J4.6
- new net N$20: J4.7
- new net N$21: J4.8
- new net N$5: J4.4
- new net N$6: J4.5
- net +3V3: now also J3.2
- net +5V: now also J4.2
- net A0: now also J3.8
- net A1: now also J3.7
- net A4/LED: now also J3.3
- net B2: now also J3.6
- net B3: now also J3.5
- net B4/USER: now also J3.4
- net GND: now also J3.1, J4.1
Changed lines of the file:
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@@
 <contactref element="R2" pad="2"/>
 <contactref element="R4" pad="2"/>
+<contactref element="J3" pad="2"/>
 <wire x1="-39.84" y1="-800" x2="-52.54" y2="-700" width="0" layer="19" extent="1-1"/>
 <wire x1="-3.81" y1="-846.19" x2="-39.84" y2="-800" width="0" layer="19" extent="1-1"/>
@@
 <wire x1="-51.27" y1="-150" x2="-51.27" y2="-250" width="0" layer="19" extent="1-1"/>
 <wire x1="-48.73" y1="-50" x2="-51.27" y2="-150" width="0" layer="19" extent="1-1"/>
+<wire x1="-48.26" y1="-990.6" x2="13.97" y2="-853.81" width="0" layer="19" extent="1-1"/>
 </signal>
 <signal name="+5V">
@@
 <contactref element="U$2" pad="2"/>
 <contactref element="U$4" pad="15"/>
+<contactref element="J4" pad="2"/>
 <wire x1="-44.9" y1="51.6" x2="-50" y2="-100" width="0" layer="19" extent="1-1"/>
 <wire x1="16.51" y1="-846.19" x2="-50" y2="-100" width="0" layer="19" extent="1-1"/>
+<wire x1="-48.26" y1="-1016" x2="16.51" y2="-846.19" width="0" layer="19" extent="1-1"/>
 </signal>
 <signal name="GND">
@@
 <contactref element="R3" pad="1"/>
 <contactref element="USER" pad="2"/>
+<contactref element="J3" pad="1"/>
+<contactref element="J4" pad="1"/>
 <wire x1="-48.26" y1="-939.8" x2="-48.26" y2="-965.2" width="0" layer="19" extent="1-1"/>
+<wire x1="-50.8" y1="-990.6" x2="-48.26" y2="-965.2" width="0" layer="19" extent="1-1"/>
+<wire x1="-50.8" y1="-1016" x2="-50.8" y2="-990.6" width="0" layer="19" extent="1-1"/>
 <wire x1="-52.54" y1="-900" x2="-48.26" y2="-939.8" width="0" layer="19" extent="1-1"/>
 <wire x1="-13.97" y1="-846.19" x2="-52.54" y2="-900" width="0" layer="19" extent="1-1"/>
@@
 <signal name="A0">
 <contactref element="U$4" pad="2"/>
+<contactref element="J3" pad="8"/>
+<wire x1="-33.02" y1="-990.6" x2="-13.97" y2="-853.81" width="0" layer="19" extent="1-1"/>
 </signal>
 <signal name="A1">
 <contactref element="U$4" pad="3"/>
+<contactref element="J3" pad="7"/>
+<wire x1="-35.56" y1="-990.6" x2="-11.43" y2="-853.81" width="0" layer="19" extent="1-1"/>
 </signal>
 <signal name="B2">
 <contactref element="U$4" pad="6"/>
+<contactref element="J3" pad="6"/>
+<wire x1="-38.1" y1="-990.6" x2="-3.81" y2="-853.81" width="0" layer="19" extent="1-1"/>
 </signal>
 <signal name="B3">
 <contactref element="U$4" pad="7"/>
+<contactref element="J3" pad="5"/>
+<wire x1="-40.64" y1="-990.6" x2="-1.27" y2="-853.81" width="0" layer="19" extent="1-1"/>
 </signal>
 <signal name="N$7">
@@
 <contactref element="R4" pad="1"/>
 <contactref element="USER" pad="1"/>
+<contactref element="J3" pad="4"/>
 <wire x1="8.89" y1="-853.81" x2="-55.08" y2="-550" width="0" layer="19" extent="1-1"/>
 <wire x1="-53.34" y1="-965.2" x2="8.89" y2="-853.81" width="0" layer="19" extent="1-1"/>
+<wire x1="-43.18" y1="-990.6" x2="-53.34" y2="-965.2" width="0" layer="19" extent="1-1"/>
 </signal>
 <signal name="A4/LED">
 <contactref element="U$4" pad="12"/>
 <contactref element="LED2" pad="A"/>
+<contactref element="J3" pad="3"/>
 <wire x1="11.43" y1="-853.81" x2="-51.27" y2="-650" width="0" layer="19" extent="1-1"/>
+<wire x1="-45.72" y1="-990.6" x2="11.43" y2="-853.81" width="0" layer="19" extent="1-1"/>
 </signal>
 <signal name="B15">
@@
 <wire x1="-44.92" y1="-500" x2="-48.73" y2="-650" width="0" layer="19" extent="1-1"/>
 </signal>
+<signal name="N$18">
+<contactref element="J4" pad="3"/>
+</signal>
+<signal name="N$5">
+<contactref element="J4" pad="4"/>
+</signal>
+<signal name="N$6">
+<contactref element="J4" pad="5"/>
+</signal>
+<signal name="N$19">
+<contactref element="J4" pad="6"/>
+</signal>
+<signal name="N$20">
+<contactref element="J4" pad="7"/>
+</signal>
+<signal name="N$21">
+<contactref element="J4" pad="8"/>
+</signal>
 </signals>

Commit message: schematic finished
Parts:
- moved J3 998.4 mm to (73.7, 0.00)
- moved J4 998.4 mm to (73.7, -25.4)
- moved USER 998.4 mm to (73.7, 25.4)
- moved RESET 998.4 mm to (73.7, 50.8)
- moved U$5 998.2 mm to (66.0, 91.4)
- moved C7 879.6 mm to (26.2, 126.3)
- moved U$3 879.6 mm to (26.2, 76.3)
- moved U$4 875.8 mm to (25.4, 25.4)
- moved C6 675.0 mm to (46.5, -32.0)
- moved R4 660.8 mm to (-27.1, 110.4)
- moved LED1 532.1 mm to (46.5, -76.8)
- moved LED2 532.1 mm to (46.5, -126.8)
- moved R3 454.2 mm to (-6.82, -47.9)
- moved R2 385.2 mm to (-14.4, -66.5)
- moved R1 310.4 mm to (-6.82, -92.7)
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Connections:
- removed net N$18: J4.3
- removed net N$19: J4.6
- removed net N$20: J4.7
- removed net N$21: J4.8
- removed net N$5: J4.4
- removed net N$6: J4.5
- net B13: now also J4.6
- net B14: now also J4.7
- net B15: now also J4.8
- net B7: now also J4.3
- net B8: now also J4.4
- net B9: now also J4.5

Commit message: update board
Parts:
- C3: value 1uF -> 0.1uF
- moved LED2 129.6 mm to (39.7, 2.65)
- moved R1 103.0 mm to (21.7, 6.30), turned to 180 degrees
- moved C7 102.5 mm to (43.8, 25.3), turned to 90 degrees
- moved R4 101.0 mm to (8.98, 16.0), turned to 90 degrees
- moved U$1 85.7 mm to (13.1, 7.91)
- moved R2 84.9 mm to (5.50, 16.0), turned to 90 degrees
- moved C2 83.5 mm to (13.1, 12.2), turned to 180 degrees
- moved LED1 81.3 mm to (28.2, 2.49)
- moved U$5 78.9 mm to (39.0, 17.3), turned to 90 degrees
- moved C4 75.9 mm to (13.1, 4.29), turned to 180 degrees
- moved J3 74.2 mm to (1.27, 16.5), turned to 90 degrees
- moved R3 70.7 mm to (34.3, 9.65)
- moved C3 68.7 mm to (13.1, 1.59), turned to 180 degrees
- moved RESET 61.3 mm to (33.7, 4.32), turned to 90 degrees
- moved C6 58.2 mm to (38.4, 25.6), turned to 270 degrees
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Connections:
- removed net N$1: C2.1, U$1.2, U$2.3
- new net N$5: J1.VBUS, U$2.2
- net +3V3: now also U$4.28
- net +5V: now also C2.1, U$1.2, U$2.3; no longer J1.VBUS, U$2.2
Routing:
- net +3V3: track 0.00 -> 146.7 mm, vias 0 -> 2
- net N$3: track 0.00 -> 103.0 mm, vias 0 -> 3
- net B4/USER: track 0.00 -> 72.5 mm, vias 0 -> 2
- net A4/LED: track 0.00 -> 51.8 mm, vias 0 -> 1
- net +5V: track 0.00 -> 51.5 mm
- net D-: track 0.00 -> 44.6 mm, vias 0 -> 1
- net D+: track 0.00 -> 41.8 mm, vias 0 -> 1
- net A1: track 0.00 -> 29.6 mm
- net A0: track 0.00 -> 29.6 mm
- net PGD: track 0.00 -> 27.6 mm, vias 0 -> 1
- net PGC: track 0.00 -> 27.6 mm, vias 0 -> 1
- net B3: track 0.00 -> 27.5 mm
- net B2: track 0.00 -> 27.5 mm
- net ID: track 0.00 -> 25.9 mm, vias 0 -> 2
- net B15: track 0.00 -> 17.7 mm
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- added copper zone on layer 16, net GND
