File: HW2/HW2/HW2.brd (EAGLE design)
At the start: 50 x 50 mm, 22 parts, among them J1 USB-MB-H, J3 CONN8, J4 CONN8

Commit message: completed board
Connections:
- net +3V3: now also U$3.2; no longer U$3.5
- net GND: now also U$3.3; no longer U$3.1
- net N$3: now also U$3.1; no longer U$3.2
- net PGC: now also U$3.5; no longer U$3.3
Routing:
- net PGC: track 28.5 -> 32.9 mm
- net +3V3: track 145.9 -> 148.9 mm
- net PGD: track 28.0 -> 28.5 mm
Other:
- board text added: "+"
- board text added: "3.3V"
- board text added: "5V"
- board text added: "A0"
- board text added: "A1"
- board text added: "A4"
- board text added: "B13"
- board text added: "B14"
- board text added: "B15"
- board text added: "B2"
- board text added: "B3"
- board text added: "B4"
- board text added: "B7"
- board text added: "B8"
- board text added: "B9"
- board text added: "GND"
- board text added: "ME433-2018-edf249"
- board text added: "SW"
