File: HW2/HW2/HW2.sch (EAGLE design)
At the start: 14 parts, among them J1 USB-MB-H

Commit message: check in
Parts:
- added C6, C7: 10uF, HW2:CPOL-USB45181B
- added U$3: PICKIT, HW2:PICKIT
- added U$4: PIC32MX250F128B, HW2:PIC32MX250F128B
- added U$5: OSCOSC, HW2:OSCOSC
- C1, C2, C4: value (none) -> 0.1uF
- LED1: value (none) -> RED
- LED2: value (none) -> GREEN
- R1: value (none) -> 330
Connections:
- new net A0: U$4.2.A0
- new net A1: U$4.3.A1
- new net A4/LED: U$4.12.A4
- new net B2: U$4.6.B2
- new net B3: U$4.7.B3
- new net B4/USER: U$4.11.B4
- new net D+: J1.D+
- new net D-: J1.D-
- new net ID: J1.ID, U$4.14.USBID/B5
- new net N$3: U$3.MCLR, U$4.1.MCLR
- new net N$7: U$4.9.OSC1, U$5.OSC2
- new net N$9: U$4.10.OSC2, U$5.OSC1
- new net PGC: U$3.PGC, U$4.5.PGEC1/B1
- new net PGD: U$3.PGD, U$4.4.PGED1/B0
- net +3V3: now also C4.1, C6.+, U$3.VDD, U$4.13.VDD
- net +5V: now also U$4.15.VBUS
- net GND: now also C1.2, C4.2, C6.-, U$3.GND, U$4.8.VSS, U$5.GND
Other:
- moved on the sheet: C1, C3, C4, C5, LED1, LED2, R1

Commit message: schem update
Parts:
- removed C5: (no value), HW2:C-US025-025X050
- added RESET, U$6: PB, HW2:PB
- C3: value (none) -> 1uF
- R2: value (none) -> 10k
Connections:
- new net B13: U$4.24.B13
- new net B14: U$4.25.B14
- new net B15: U$4.26..B15
- new net B7: U$4.16.B7
- new net B8: U$4.17.B8
- new net B9: U$4.18.B9
- new net N$13: C7.+, U$4.20.VCAP
- new net N$4: LED2.C, R3.2
- net +3V3: now also C3.1, R2.2, U$4.23.VUSB3V3
- net A4/LED: now also LED2.A
- net D+: now also U$4.21.D+/B10
- net D-: now also U$4.22.D-/B11
- net GND: now also C3.2, C7.-, R3.1, RESET.2, U$4.19.VSS, U$4.27.AVSS
- net N$3: now also R2.1, RESET.1
Other:
- moved on the sheet: C3, C7, LED2, R2, R3, R4

Commit message: another update
Parts:
- removed U$6: PB, HW2:PB
- added J3, J4: CONN8, HW2:CONN8
- added USER: PB, HW2:PB
- R3: value (none) -> 330
- R4: value (none) -> 10k
Connections:
- net +3V3: now also R4.2
- net B4/USER: now also R4.1, USER.1
- net GND: now also USER.2
Changed lines of the file:
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@@
 <part name="R1" library="HW2" deviceset="R-US_" device="0207/10" package3d_urn="urn:adsk.eagle:package:25939/1" value="330"/>
 <part name="R2" library="HW2" deviceset="R-US_" device="0207/10" package3d_urn="urn:adsk.eagle:package:25939/1" value="10k"/>
-<part name="R3" library="HW2" deviceset="R-US_" device="0207/10" package3d_urn="urn:adsk.eagle:package:25939/1"/>
-<part name="R4" library="HW2" deviceset="R-US_" device="0207/10" package3d_urn="urn:adsk.eagle:package:25939/1"/>
+<part name="R3" library="HW2" deviceset="R-US_" device="0207/10" package3d_urn="urn:adsk.eagle:package:25939/1" value="330"/>
+<part name="R4" library="HW2" deviceset="R-US_" device="0207/10" package3d_urn="urn:adsk.eagle:package:25939/1" value="10k"/>
 <part name="GND3" library="HW2" deviceset="GND" device=""/>
 <part name="GND4" library="HW2" deviceset="GND" device=""/>
@@
 <part name="GND15" library="HW2" deviceset="GND" device=""/>
 <part name="GND16" library="HW2" deviceset="GND" device=""/>
-<part name="U$6" library="HW2" deviceset="PB" device=""/>
+<part name="USER" library="HW2" deviceset="PB" device=""/>
 <part name="+3V7" library="HW2" deviceset="+3V3" device=""/>
+<part name="J3" library="HW2" deviceset="CONN8" device=""/>
+<part name="J4" library="HW2" deviceset="CONN8" device=""/>
 </parts>
 <sheets>
@@
 <instance part="GND14" gate="1" x="63.5" y="-33.02"/>
 <instance part="GND15" gate="1" x="119.38" y="0"/>
-<instance part="GND16" gate="1" x="124.46" y="-35.56"/>
-<instance part="U$6" gate="G$1" x="149.86" y="-33.02" rot="R270"/>
-<instance part="+3V7" gate="G$1" x="144.78" y="0"/>
+<instance part="GND16" gate="1" x="124.46" y="-33.02"/>
+<instance part="USER" gate="G$1" x="139.7" y="-20.32" smashed="yes" rot="R270">
+<attribute name="NAME" x="144.78" y="-12.7" size="1.778" layer="94"/>
+<attribute name="VALUE" x="144.78" y="-27.94" size="1.778" layer="94"/>
+</instance>
+<instance part="+3V7" gate="G$1" x="124.46" y="-10.16"/>
+<instance part="J3" gate="G$1" x="139.7" y="-71.12" rot="MR0"/>
+<instance part="J4" gate="G$1" x="152.4" y="-71.12"/>
 </instances>
 <busses>
@@
 <pinref part="+3V6" gate="G$1" pin="+3V3"/>
 </segment>
+<segment>
+<pinref part="R4" gate="G$1" pin="2"/>
+<pinref part="+3V7" gate="G$1" pin="+3V3"/>
+</segment>
 </net>
 <net name="+5V" class="0">
@@
 <pinref part="R3" gate="G$1" pin="1"/>
 <pinref part="GND15" gate="1" pin="GND"/>
+</segment>
+<segment>
+<pinref part="USER" gate="G$1" pin="2"/>
+<wire x1="139.7" y1="-30.48" x2="124.46" y2="-30.48" width="0.1524" layer="91"/>
+<pinref part="GND16" gate="1" pin="GND"/>
 </segment>
 </net>
@@
 <label x="35.56" y="-96.52" size="1.778" layer="95"/>
 </segment>
-</net>
+<segment>
+<pinref part="R4" gate="G$1" pin="1"/>
+<wire x1="124.46" y1="-22.86" x2="132.08" y2="-22.86" width="0.1524" layer="91"/>
+<pinref part="USER" gate="G$1" pin="1"/>
+<wire x1="132.08" y1="-22.86" x2="132.08" y2="-10.16" width="0.1524" layer="91"/>
+<wire x1="132.08" y1="-10.16" x2="139.7" y2="-10.16" width="0.1524" layer="91"/>
+<wire x1="124.46" y1="-22.86" x2="101.6" y2="-22.86" width="0.1524" layer="91"/>
+<junction x="124.46" y="-22.86"/>
+<label x="101.6" y="-22.86" size="1.778" layer="95"/>
+</segment>
+</net>

Commit message: sign on
Connections:
- new net N$18: J4.3
- new net N$19: J4.6
- new net N$20: J4.7
- new net N$21: J4.8
- new net N$5: J4.4
- new net N$6: J4.5
- net +3V3: now also J3.2
- net +5V: now also J4.2
- net A0: now also J3.8
- net A1: now also J3.7
- net A4/LED: now also J3.3
- net B2: now also J3.6
- net B3: now also J3.5
- net B4/USER: now also J3.4
- net GND: now also J3.1, J4.1
Changed lines of the file:
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@@
 <part name="J3" library="HW2" deviceset="CONN8" device=""/>
 <part name="J4" library="HW2" deviceset="CONN8" device=""/>
+<part name="GND17" library="HW2" deviceset="GND" device=""/>
+<part name="GND18" library="HW2" deviceset="GND" device=""/>
+<part name="+3V8" library="HW2" deviceset="+3V3" device=""/>
+<part name="P+3" library="HW2" deviceset="+5V" device=""/>
 </parts>
 <sheets>
@@
 <instance part="J3" gate="G$1" x="139.7" y="-71.12" rot="MR0"/>
 <instance part="J4" gate="G$1" x="152.4" y="-71.12"/>
+<instance part="GND17" gate="1" x="129.54" y="-86.36"/>
+<instance part="GND18" gate="1" x="162.56" y="-86.36"/>
+<instance part="+3V8" gate="G$1" x="121.92" y="-81.28" rot="R180"/>
+<instance part="P+3" gate="1" x="170.18" y="-81.28" rot="R180"/>
 </instances>
 <busses>
@@
 <pinref part="+3V7" gate="G$1" pin="+3V3"/>
 </segment>
+<segment>
+<pinref part="+3V8" gate="G$1" pin="+3V3"/>
+<pinref part="J3" gate="G$1" pin="2"/>
+<wire x1="121.92" y1="-78.74" x2="121.92" y2="-76.2" width="0.1524" layer="91"/>
+<wire x1="121.92" y1="-76.2" x2="134.62" y2="-76.2" width="0.1524" layer="91"/>
+</segment>
 </net>
 <net name="+5V" class="0">
@@
 <pinref part="P+2" gate="1" pin="+5V"/>
 </segment>
+<segment>
+<pinref part="J4" gate="G$1" pin="2"/>
+<wire x1="157.48" y1="-76.2" x2="170.18" y2="-76.2" width="0.1524" layer="91"/>
+<pinref part="P+3" gate="1" pin="+5V"/>
+<wire x1="170.18" y1="-76.2" x2="170.18" y2="-78.74" width="0.1524" layer="91"/>
+</segment>
 </net>
 <net name="GND" class="0">
@@
 <wire x1="139.7" y1="-30.48" x2="124.46" y2="-30.48" width="0.1524" layer="91"/>
 <pinref part="GND16" gate="1" pin="GND"/>
+</segment>
+<segment>
+<pinref part="J3" gate="G$1" pin="1"/>
+<wire x1="134.62" y1="-78.74" x2="129.54" y2="-78.74" width="0.1524" layer="91"/>
+<wire x1="129.54" y1="-78.74" x2="129.54" y2="-83.82" width="0.1524" layer="91"/>
+<pinref part="GND17" gate="1" pin="GND"/>
+</segment>
+<segment>
+<pinref part="J4" gate="G$1" pin="1"/>
+<wire x1="157.48" y1="-78.74" x2="162.56" y2="-78.74" width="0.1524" layer="91"/>
+<wire x1="162.56" y1="-78.74" x2="162.56" y2="-83.82" width="0.1524" layer="91"/>
+<pinref part="GND18" gate="1" pin="GND"/>
 </segment>
 </net>
@@
 <wire x1="45.72" y1="-50.8" x2="33.02" y2="-50.8" width="0.1524" layer="91"/>
 </segment>
+<segment>
+<pinref part="J3" gate="G$1" pin="8"/>
+<wire x1="134.62" y1="-60.96" x2="121.92" y2="-60.96" width="0.1524" layer="91"/>
+<label x="121.92" y="-60.96" size="1.778" layer="95"/>
+</segment>
 </net>
 <net name="A1" class="0">
@@
 <wire x1="45.72" y1="-55.88" x2="33.02" y2="-55.88" width="0.1524" layer="91"/>
 <label x="33.02" y="-55.88" size="1.778" layer="95"/>
+</segment>
+<segment>
+<pinref part="J3" gate="G$1" pin="7"/>
+<wire x1="134.62" y1="-63.5" x2="121.92" y2="-63.5" width="0.1524" layer="91"/>
+<label x="121.92" y="-63.5" size="1.778" layer="95"/>
 </segment>
 </net>
@@
 <label x="33.02" y="-71.12" size="1.778" layer="95"/>
 </segment>
+<segment>
+<pinref part="J3" gate="G$1" pin="6"/>
+<wire x1="134.62" y1="-66.04" x2="121.92" y2="-66.04" width="0.1524" layer="91"/>
+<label x="121.92" y="-66.04" size="1.778" layer="95"/>
+</segment>
 </net>
 <net name="B3" class="0">
@@
 <wire x1="45.72" y1="-76.2" x2="33.02" y2="-76.2" width="0.1524" layer="91"/>
 <label x="33.02" y="-76.2" size="1.778" layer="95"/>
+</segment>
+<segment>
+<pinref part="J3" gate="G$1" pin="5"/>
+<wire x1="134.62" y1="-68.58" x2="121.92" y2="-68.58" width="0.1524" layer="91"/>
+<label x="121.92" y="-68.58" size="1.778" layer="95"/>
 </segment>
 </net>
@@
 <label x="101.6" y="-22.86" size="1.778" layer="95"/>
 </segment>
+<segment>
+<pinref part="J3" gate="G$1" pin="4"/>
+<wire x1="134.62" y1="-71.12" x2="121.92" y2="-71.12" width="0.1524" layer="91"/>
+<label x="121.92" y="-71.12" size="1.778" layer="95"/>
+</segment>
 </net>
 <net name="A4/LED" class="0">
@@
 <wire x1="119.38" y1="20.32" x2="119.38" y2="35.56" width="0.1524" layer="91"/>
 <label x="116.84" y="35.56" size="1.778" layer="95"/>
+</segment>
+<segment>
+<pinref part="J3" gate="G$1" pin="3"/>
+<wire x1="134.62" y1="-73.66" x2="121.92" y2="-73.66" width="0.1524" layer="91"/>
+<label x="121.92" y="-73.66" size="1.778" layer="95"/>
 </segment>
 </net>
@@
 </segment>
 </net>
+<net name="N$18" class="0">
+<segment>
+<pinref part="J4" gate="G$1" pin="3"/>
+<wire x1="157.48" y1="-73.66" x2="170.18" y2="-73.66" width="0.1524" layer="91"/>
+</segment>
+</net>
+<net name="N$5" class="0">
+<segment>
+<pinref part="J4" gate="G$1" pin="4"/>
+<wire x1="157.48" y1="-71.12" x2="170.18" y2="-71.12" width="0.1524" layer="91"/>
+</segment>
+</net>
+<net name="N$6" class="0">
+<segment>
+<pinref part="J4" gate="G$1" pin="5"/>
+<wire x1="157.48" y1="-68.58" x2="170.18" y2="-68.58" width="0.1524" layer="91"/>
+</segment>
+</net>
+<net name="N$19" class="0">
+<segment>
+<pinref part="J4" gate="G$1" pin="6"/>
+<wire x1="157.48" y1="-66.04" x2="170.18" y2="-66.04" width="0.1524" layer="91"/>
+</segment>
+</net>
+<net name="N$20" class="0">
+<segment>
+<pinref part="J4" gate="G$1" pin="7"/>
+<wire x1="157.48" y1="-63.5" x2="170.18" y2="-63.5" width="0.1524" layer="91"/>
+</segment>
+</net>
+<net name="N$21" class="0">
+<segment>
+<pinref part="J4" gate="G$1" pin="8"/>
+<wire x1="157.48" y1="-60.96" x2="170.18" y2="-60.96" width="0.1524" layer="91"/>
+</segment>
+</net>

Commit message: schematic finished
Connections:
- removed net N$18: J4.3
- removed net N$19: J4.6
- removed net N$20: J4.7
- removed net N$21: J4.8
- removed net N$5: J4.4
- removed net N$6: J4.5
- net B13: now also J4.6
- net B14: now also J4.7
- net B15: now also J4.8
- net B7: now also J4.3
- net B8: now also J4.4
- net B9: now also J4.5
Changed lines of the file:
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@@
 <label x="96.52" y="-55.88" size="1.778" layer="95"/>
+</segment>
+<segment>
+<pinref part="J4" gate="G$1" pin="8"/>
+<wire x1="157.48" y1="-60.96" x2="170.18" y2="-60.96" width="0.1524" layer="91"/>
+<label x="167.64" y="-60.96" size="1.778" layer="95"/>
 </segment>
 </net>
@@
 <label x="96.52" y="-60.96" size="1.778" layer="95"/>
 </segment>
+<segment>
+<pinref part="J4" gate="G$1" pin="7"/>
+<wire x1="157.48" y1="-63.5" x2="170.18" y2="-63.5" width="0.1524" layer="91"/>
+<label x="167.64" y="-63.5" size="1.778" layer="95"/>
+</segment>
 </net>
 <net name="B13" class="0">
@@
 <wire x1="86.36" y1="-66.04" x2="99.06" y2="-66.04" width="0.1524" layer="91"/>
 <label x="96.52" y="-66.04" size="1.778" layer="95"/>
+</segment>
+<segment>
+<pinref part="J4" gate="G$1" pin="6"/>
+<wire x1="157.48" y1="-66.04" x2="170.18" y2="-66.04" width="0.1524" layer="91"/>
+<label x="167.64" y="-66.04" size="1.778" layer="95"/>
 </segment>
 </net>
@@
 <label x="96.52" y="-96.52" size="1.778" layer="95"/>
 </segment>
+<segment>
+<pinref part="J4" gate="G$1" pin="5"/>
+<wire x1="157.48" y1="-68.58" x2="170.18" y2="-68.58" width="0.1524" layer="91"/>
+<label x="167.64" y="-68.58" size="1.778" layer="95"/>
+</segment>
 </net>
 <net name="B8" class="0">
@@
 <wire x1="86.36" y1="-101.6" x2="99.06" y2="-101.6" width="0.1524" layer="91"/>
 <label x="96.52" y="-101.6" size="1.778" layer="95"/>
+</segment>
+<segment>
+<pinref part="J4" gate="G$1" pin="4"/>
+<wire x1="157.48" y1="-71.12" x2="170.18" y2="-71.12" width="0.1524" layer="91"/>
+<label x="167.64" y="-71.12" size="1.778" layer="95"/>
 </segment>
 </net>
@@
 <label x="96.52" y="-106.68" size="1.778" layer="95"/>
 </segment>
+<segment>
+<pinref part="J4" gate="G$1" pin="3"/>
+<wire x1="157.48" y1="-73.66" x2="170.18" y2="-73.66" width="0.1524" layer="91"/>
+<label x="167.64" y="-73.66" size="1.778" layer="95"/>
+</segment>
 </net>
 <net name="N$4" class="0">
@@
 </segment>
 </net>
-<net name="N$18" class="0">
-<segment>
-<pinref part="J4" gate="G$1" pin="3"/>
-<wire x1="157.48" y1="-73.66" x2="170.18" y2="-73.66" width="0.1524" layer="91"/>
-</segment>
-</net>
-<net name="N$5" class="0">
-<segment>
-<pinref part="J4" gate="G$1" pin="4"/>
-<wire x1="157.48" y1="-71.12" x2="170.18" y2="-71.12" width="0.1524" layer="91"/>
-</segment>
-</net>
-<net name="N$6" class="0">
-<segment>
-<pinref part="J4" gate="G$1" pin="5"/>
-<wire x1="157.48" y1="-68.58" x2="170.18" y2="-68.58" width="0.1524" layer="91"/>
-</segment>
-</net>
-<net name="N$19" class="0">
-<segment>
-<pinref part="J4" gate="G$1" pin="6"/>
-<wire x1="157.48" y1="-66.04" x2="170.18" y2="-66.04" width="0.1524" layer="91"/>
-</segment>
-</net>
-<net name="N$20" class="0">
-<segment>
-<pinref part="J4" gate="G$1" pin="7"/>
-<wire x1="157.48" y1="-63.5" x2="170.18" y2="-63.5" width="0.1524" layer="91"/>
-</segment>
-</net>
-<net name="N$21" class="0">
-<segment>
-<pinref part="J4" gate="G$1" pin="8"/>
-<wire x1="157.48" y1="-60.96" x2="170.18" y2="-60.96" width="0.1524" layer="91"/>
-</segment>
-</net>

Commit message: update board
Parts:
- C3: value 1uF -> 0.1uF
Connections:
- removed net N$1: C2.1, U$1.2.VIN, U$2.3
- new net N$5: J1.VBUS, U$2.2
- net +3V3: now also U$4.28.AVDD
- net +5V: now also C2.1, U$1.2.VIN, U$2.3; no longer J1.VBUS, U$2.2
Changed lines of the file:
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@@
 <part name="U$1" library="HW2" deviceset="MCP1702" device=""/>
 <part name="+3V1" library="HW2" deviceset="+3V3" device=""/>
-<part name="P+1" library="HW2" deviceset="+5V" device=""/>
 <part name="GND1" library="HW2" deviceset="GND" device=""/>
 <part name="GND2" library="HW2" deviceset="GND" device=""/>
@@
 <part name="C1" library="HW2" deviceset="C-US" device="025-025X050" package3d_urn="urn:adsk.eagle:package:26151/1" value="0.1uF"/>
 <part name="C2" library="HW2" deviceset="C-US" device="025-025X050" package3d_urn="urn:adsk.eagle:package:26151/1" value="0.1uF"/>
-<part name="C3" library="HW2" deviceset="C-US" device="025-025X050" package3d_urn="urn:adsk.eagle:package:26151/1" value="1uF"/>
+<part name="C3" library="HW2" deviceset="C-US" device="025-025X050" package3d_urn="urn:adsk.eagle:package:26151/1" value="0.1uF"/>
 <part name="C4" library="HW2" deviceset="C-US" device="025-025X050" package3d_urn="urn:adsk.eagle:package:26151/1" value="0.1uF"/>
 <part name="R1" library="HW2" deviceset="R-US_" device="0207/10" package3d_urn="urn:adsk.eagle:package:25939/1" value="330"/>
@@
 <part name="+3V8" library="HW2" deviceset="+3V3" device=""/>
 <part name="P+3" library="HW2" deviceset="+5V" device=""/>
+<part name="P+1" library="HW2" deviceset="+5V" device=""/>
 </parts>
 <sheets>
@@
 <instance part="U$1" gate="G$1" x="12.7" y="22.86" rot="R90"/>
 <instance part="+3V1" gate="G$1" x="58.42" y="43.18" rot="R270"/>
-<instance part="P+1" gate="1" x="76.2" y="35.56"/>
 <instance part="GND1" gate="1" x="91.44" y="15.24"/>
 <instance part="GND2" gate="1" x="33.02" y="15.24"/>
@@
 <instance part="R4" gate="G$1" x="124.46" y="-17.78" rot="R90"/>
 <instance part="GND3" gate="1" x="38.1" y="33.02"/>
-<instance part="GND4" gate="1" x="25.4" y="-7.62"/>
+<instance part="GND4" gate="1" x="25.4" y="-12.7"/>
 <instance part="LED1" gate="G$1" x="53.34" y="30.48" smashed="yes" rot="R90">
 <attribute name="NAME" x="57.912" y="34.036" size="1.778" layer="95" rot="R180"/>
@@
 <instance part="+3V8" gate="G$1" x="121.92" y="-81.28" rot="R180"/>
 <instance part="P+3" gate="1" x="170.18" y="-81.28" rot="R180"/>
+<instance part="P+1" gate="1" x="35.56" y="-7.62" rot="R180"/>
 </instances>
 <busses>
@@
 </segment>
 <segment>
-<wire x1="101.6" y1="-45.72" x2="86.36" y2="-45.72" width="0.1524" layer="91"/>
 <wire x1="101.6" y1="-45.72" x2="101.6" y2="-43.18" width="0.1524" layer="91"/>
 <pinref part="C3" gate="G$1" pin="1"/>
@@
 <wire x1="104.14" y1="-43.18" x2="111.76" y2="-43.18" width="0.1524" layer="91"/>
 <junction x="104.14" y="-43.18"/>
+<pinref part="U$4" gate="G$1" pin="28.AVDD"/>
+<wire x1="86.36" y1="-45.72" x2="101.6" y2="-45.72" width="0.1524" layer="91"/>
 </segment>
 <segment>
@@
 <net name="+5V" class="0">
 <segment>
-<pinref part="J1" gate="G$1" pin="VBUS"/>
-<wire x1="76.2" y1="27.94" x2="93.98" y2="27.94" width="0.1524" layer="91"/>
-<pinref part="P+1" gate="1" pin="+5V"/>
-<wire x1="76.2" y1="27.94" x2="76.2" y2="33.02" width="0.1524" layer="91"/>
-<wire x1="76.2" y1="25.4" x2="76.2" y2="27.94" width="0.1524" layer="91"/>
-<junction x="76.2" y="27.94"/>
-<pinref part="U$2" gate="G$1" pin="2"/>
-<wire x1="58.42" y1="20.32" x2="58.42" y2="25.4" width="0.1524" layer="91"/>
-<wire x1="58.42" y1="25.4" x2="76.2" y2="25.4" width="0.1524" layer="91"/>
-</segment>
-<segment>
 <pinref part="U$4" gate="G$1" pin="15.VBUS"/>
 <wire x1="86.36" y1="-111.76" x2="101.6" y2="-111.76" width="0.1524" layer="91"/>
@@
 <wire x1="170.18" y1="-76.2" x2="170.18" y2="-78.74" width="0.1524" layer="91"/>
 </segment>
+<segment>
+<pinref part="U$1" gate="G$1" pin="2.VIN"/>
+<wire x1="12.7" y1="7.62" x2="12.7" y2="2.54" width="0.1524" layer="91"/>
+<wire x1="12.7" y1="2.54" x2="25.4" y2="2.54" width="0.1524" layer="91"/>
+<wire x1="25.4" y1="2.54" x2="35.56" y2="2.54" width="0.1524" layer="91"/>
+<wire x1="35.56" y1="2.54" x2="35.56" y2="-5.08" width="0.1524" layer="91"/>
+<pinref part="C2" gate="G$1" pin="1"/>
+<wire x1="25.4" y1="0" x2="25.4" y2="2.54" width="0.1524" layer="91"/>
+<junction x="25.4" y="2.54"/>
+<pinref part="P+1" gate="1" pin="+5V"/>
+<wire x1="35.56" y1="2.54" x2="35.56" y2="10.16" width="0.1524" layer="91"/>
+<junction x="35.56" y="2.54"/>
+<pinref part="U$2" gate="G$1" pin="3"/>
+<wire x1="53.34" y1="25.4" x2="53.34" y2="20.32" width="0.1524" layer="91"/>
+<wire x1="43.18" y1="25.4" x2="53.34" y2="25.4" width="0.1524" layer="91"/>
+<wire x1="43.18" y1="10.16" x2="43.18" y2="25.4" width="0.1524" layer="91"/>
+<wire x1="35.56" y1="10.16" x2="43.18" y2="10.16" width="0.1524" layer="91"/>
+</segment>
 </net>
 <net name="GND" class="0">
@@
 <pinref part="C2" gate="G$1" pin="2"/>
 <pinref part="GND4" gate="1" pin="GND"/>
-<wire x1="25.4" y1="-5.08" x2="25.4" y2="-7.62" width="0.1524" layer="91"/>
+<wire x1="25.4" y1="-10.16" x2="25.4" y2="-7.62" width="0.1524" layer="91"/>
 </segment>
 <segment>
@@
 <wire x1="162.56" y1="-78.74" x2="162.56" y2="-83.82" width="0.1524" layer="91"/>
 <pinref part="GND18" gate="1" pin="GND"/>
-</segment>
-</net>
-<net name="N$1" class="0">
-<segment>
-<pinref part="U$1" gate="G$1" pin="2.VIN"/>
-<wire x1="12.7" y1="7.62" x2="12.7" y2="2.54" width="0.1524" layer="91"/>
-<wire x1="12.7" y1="2.54" x2="25.4" y2="2.54" width="0.1524" layer="91"/>
-<wire x1="25.4" y1="2.54" x2="35.56" y2="2.54" width="0.1524" layer="91"/>
-<wire x1="35.56" y1="2.54" x2="35.56" y2="10.16" width="0.1524" layer="91"/>
-<wire x1="35.56" y1="10.16" x2="43.18" y2="10.16" width="0.1524" layer="91"/>
-<wire x1="43.18" y1="10.16" x2="43.18" y2="25.4" width="0.1524" layer="91"/>
-<wire x1="43.18" y1="25.4" x2="53.34" y2="25.4" width="0.1524" layer="91"/>
-<pinref part="U$2" gate="G$1" pin="3"/>
-<wire x1="53.34" y1="25.4" x2="53.34" y2="20.32" width="0.1524" layer="91"/>
-<pinref part="C2" gate="G$1" pin="1"/>
-<wire x1="25.4" y1="0" x2="25.4" y2="2.54" width="0.1524" layer="91"/>
-<junction x="25.4" y="2.54"/>
 </segment>
 </net>
@@
 <net name="A0" class="0">
 <segment>
+<pinref part="J3" gate="G$1" pin="8"/>
+<wire x1="134.62" y1="-60.96" x2="121.92" y2="-60.96" width="0.1524" layer="91"/>
+<label x="121.92" y="-60.96" size="1.778" layer="95"/>
+</segment>
+<segment>
 <pinref part="U$4" gate="G$1" pin="2.A0"/>
 <wire x1="45.72" y1="-50.8" x2="33.02" y2="-50.8" width="0.1524" layer="91"/>
 <label x="33.02" y="-50.8" size="1.778" layer="95"/>
-<wire x1="45.72" y1="-50.8" x2="33.02" y2="-50.8" width="0.1524" layer="91"/>
-</segment>
-<segment>
-<pinref part="J3" gate="G$1" pin="8"/>
-<wire x1="134.62" y1="-60.96" x2="121.92" y2="-60.96" width="0.1524" layer="91"/>
-<label x="121.92" y="-60.96" size="1.778" layer="95"/>
 </segment>
 </net>
@@
 <net name="B2" class="0">
 <segment>
-<pinref part="U$4" gate="G$1" pin="6.B2"/>
-<wire x1="45.72" y1="-71.12" x2="33.02" y2="-71.12" width="0.1524" layer="91"/>
-<wire x1="45.72" y1="-71.12" x2="33.02" y2="-71.12" width="0.1524" layer="91"/>
-<label x="33.02" y="-71.12" size="1.778" layer="95"/>
-</segment>
-<segment>
 <pinref part="J3" gate="G$1" pin="6"/>
 <wire x1="134.62" y1="-66.04" x2="121.92" y2="-66.04" width="0.1524" layer="91"/>
 <label x="121.92" y="-66.04" size="1.778" layer="95"/>
 </segment>
+<segment>
+<pinref part="U$4" gate="G$1" pin="6.B2"/>
+<wire x1="45.72" y1="-71.12" x2="33.02" y2="-71.12" width="0.1524" layer="91"/>
+<label x="33.02" y="-71.12" size="1.778" layer="95"/>
+</segment>
 </net>
 <net name="B3" class="0">
-<segment>
-<pinref part="U$4" gate="G$1" pin="7.B3"/>
-<wire x1="45.72" y1="-76.2" x2="33.02" y2="-76.2" width="0.1524" layer="91"/>
-<wire x1="45.72" y1="-76.2" x2="33.02" y2="-76.2" width="0.1524" layer="91"/>
-<label x="33.02" y="-76.2" size="1.778" layer="95"/>
-</segment>
 <segment>
 <pinref part="J3" gate="G$1" pin="5"/>
 <wire x1="134.62" y1="-68.58" x2="121.92" y2="-68.58" width="0.1524" layer="91"/>
 <label x="121.92" y="-68.58" size="1.778" layer="95"/>
+</segment>
+<segment>
+<pinref part="U$4" gate="G$1" pin="7.B3"/>
+<wire x1="45.72" y1="-76.2" x2="33.02" y2="-76.2" width="0.1524" layer="91"/>
 </segment>
 </net>
@@
 </segment>
 </net>
+<net name="N$5" class="0">
+<segment>
+<pinref part="J1" gate="G$1" pin="VBUS"/>
+<wire x1="76.2" y1="27.94" x2="93.98" y2="27.94" width="0.1524" layer="91"/>
+<wire x1="76.2" y1="25.4" x2="76.2" y2="27.94" width="0.1524" layer="91"/>
+<pinref part="U$2" gate="G$1" pin="2"/>
+<wire x1="58.42" y1="20.32" x2="58.42" y2="25.4" width="0.1524" layer="91"/>
+<wire x1="58.42" y1="25.4" x2="76.2" y2="25.4" width="0.1524" layer="91"/>
+</segment>
+</net>
