File: HW2/HW2/HW2.sch (EAGLE design)
At the start: 22 parts, among them J1 USB-MB-H, J3 CONN8, J4 CONN8

Commit message: completed board
Changed lines of the file:
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@@
 <instance part="U$3" gate="G$1" x="25.4" y="-35.56" rot="R180"/>
 <instance part="U$4" gate="G$1" x="76.2" y="-78.74"/>
-<instance part="+3V2" gate="G$1" x="33.02" y="-40.64" smashed="yes" rot="R270">
-<attribute name="VALUE" x="30.48" y="-43.18" size="1.778" layer="96"/>
+<instance part="+3V2" gate="G$1" x="30.48" y="-40.64" smashed="yes" rot="R270">
+<attribute name="VALUE" x="27.94" y="-43.18" size="1.778" layer="96"/>
 </instance>
 <instance part="GND7" gate="1" x="40.64" y="-40.64"/>
@@
 <segment>
 <pinref part="U$3" gate="G$1" pin="VDD"/>
-<wire x1="25.4" y1="-40.64" x2="30.48" y2="-40.64" width="0.1524" layer="91"/>
+<wire x1="25.4" y1="-40.64" x2="27.94" y2="-40.64" width="0.1524" layer="91"/>
 <pinref part="+3V2" gate="G$1" pin="+3V3"/>
 </segment>
